File: EAGLE/DIP_rev_C/FX-Flash_DIP_rev_C.sch (EAGLE design)
At the start: 6 parts, among them IC1 SST39SF040-70-4C-PHE, IC2 SN74LVC32ADR

Commit message: Update DIP design to use 0805 capacitors for easy soldering (rev C)
Parts:
- C1, C2: device PC-Engine0402:C-USC0402 -> resistor:C-USC0805
Changed lines of the file:
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@@
 <part name="U$2" library="PC-Engine" deviceset="FXCARD-EDGE" device=""/>
 <part name="IC2" library="PC-Engine" deviceset="SN74LVC32ADR" device=""/>
-<part name="C1" library="PC-Engine0402" deviceset="C-US" device="C0402" package3d_urn="urn:adsk.eagle:package:23626/2" value="100nF"/>
-<part name="C2" library="PC-Engine0402" deviceset="C-US" device="C0402" package3d_urn="urn:adsk.eagle:package:23626/2" value="100nF"/>
+<part name="C1" library="resistor" library_urn="urn:adsk.eagle:library:348" deviceset="C-US" device="C0805" package3d_urn="urn:adsk.eagle:package:23617/2" value="100nF"/>
+<part name="C2" library="resistor" library_urn="urn:adsk.eagle:library:348" deviceset="C-US" device="C0805" package3d_urn="urn:adsk.eagle:package:23617/2" value="100nF"/>
 <part name="IC1" library="PC-Engine" deviceset="SST39SF040-70-4C-PHE" device=""/>
 <part name="P+1" library="supply1" library_urn="urn:adsk.eagle:library:371" deviceset="+5V" device=""/>
